File: SaTea.kicad_pcb (KiCad board)
At the start: 2 copper layers, 96.5 x 91.4 mm, 23 parts, among them J1 Conn_01x20, J2 Conn_01x20, J3 Conn_01x06, J4 Conn_01x06, J5 Conn_01x06, J6 Conn_01x06, J7 Conn_01x06, J8 Conn_01x06, SW1 SW_SPDT, U2 DC/DC 5V out

Commit message: add scheme
Parts:
- moved R1 0.64 mm to (140.3, 142.2)
- moved BT1 0.64 mm to (124.7, 124.5)
- moved R2 0.63 mm to (135.3, 142.2)
Routing:
- net +3V3: track 151.9 -> 171.0 mm, vias 6 -> 5
- net VBAT: track 47.2 -> 49.2 mm
- net /PB4: track 54.0 -> 52.3 mm
- net Net-(SC1-+): track 92.3 -> 91.3 mm
- net /PB0: track 51.5 -> 50.7 mm
- net /PA4: track 75.6 -> 76.3 mm
- net /PA6: track 57.7 -> 57.0 mm
- net Net-(D1-A): track 36.2 -> 35.6 mm
- net VSYS: track 180.9 -> 181.5 mm
- net /PA1: track 46.4 -> 45.7 mm
- net /PB1: track 48.2 -> 47.6 mm
- net /PA0: track 48.2 -> 47.7 mm
- net /PB3: track 40.0 -> 40.5 mm
- net /PA5: track 58.4 -> 57.9 mm
- net GND: vias 11 -> 12

Commit message: Update 31-12-24-NEZ-Final
Parts:
- J3, J4, J5, J6, J7, J8: value Conn_01x06 -> Conn_01x04
- U1: value ~ -> BMM
Routing:
- net /PA4: track 76.3 -> 79.5 mm
Other:
- board text added: "Sa"
- board text added: "Tea"
- board text removed: "JLCJLCJLCJLC"
