File: SaTea.kicad_sch (KiCad schematic)
At the start: 23 parts, among them J1 Conn_01x20, J2 Conn_01x20, J3 Conn_01x06, J4 Conn_01x06, J5 Conn_01x06, J6 Conn_01x06, J7 Conn_01x06, J8 Conn_01x06, SW1 SW_SPDT, U2 DC/DC 5V out

Commit message: Update 31-12-24-NEZ-Final
Parts:
- BT1: Inv. number (none) -> N/A; Mnf. number (none) -> 13400; Price (CZK) /pc (none) -> 0; Supplier (none) -> Re-Use
- D1: Inv. number (none) -> C53568; Mnf. number (none) -> 1N4007RLG; Price (CZK) /pc (none) -> 1; Supplier (none) -> LCSC
- H1, H2, JP1, JP2, JP3, JP4: Price (CZK) /pc (none) -> 0
- J1, J2: Inv. number (none) -> N/A; Mnf. number (none) -> N/A; Price (CZK) /pc (none) -> 2.17; Supplier (none) -> Ali
- J3, J4, J5, J6, J7, J8: value Conn_01x06 -> Conn_01x04; Price (CZK) /pc (none) -> 0
- R1: Inv. number (none) -> C114065; Mnf. number (none) -> RC0603FR-0722KL; Price (CZK) /pc (none) -> 0,029; Supplier (none) -> LCSC
- R2: Inv. number (none) -> C137662; Mnf. number (none) -> RC0603JR-0712KL; Price (CZK) /pc (none) -> 0,024; Supplier (none) -> LCSC
- SC1, SC2: Inv. number (none) -> N/A; Mnf. number (none) -> AK68X36; Price (CZK) /pc (none) -> 21,53; Supplier (none) -> Ali
- SW1: Inv. number (none) -> N/A; Mnf. number (none) -> SS12D00; Price (CZK) /pc (none) -> 0,94; Supplier (none) -> Ali
- U1: value ~ -> BMM; Inv. number (none) -> N/A; Mnf. number (none) -> N/A; Price (CZK) /pc (none) -> 6,28; Supplier (none) -> Ali
- U2: Inv. number (none) -> N/A; Mnf. number (none) -> N/A; Price (CZK) /pc (none) -> 7,92; Supplier (none) -> Ali
Connections:
- no-connect marks 2 -> 12
Other:
- company: (none) -> TeaTech & VoŠ a SPŠE Plzeň
- title: (none) -> SaTea - small "teachy" satellite
